File: project, schematic, and pcb files/hackpad.kicad_pcb (KiCad board)
At the start: 2 copper layers, 99.4 x 81.4 mm, 37 parts, among them J1 Conn_01x04_Pin, SW1 SW_Push, SW10 RotaryEncoder_Switch, SW11 RotaryEncoder_Switch, SW2 SW_Push, SW3 SW_Push, SW4 SW_Push, SW5 SW_Push, SW6 SW_Push, SW7 SW_Push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

Commit message: Add files via upload
Parts:
- added D10: SK6812MINI, LED_SMD:LED_SK6812MINI_PLCC4_3.5x3.5mm_P1.75mm, F.Cu at (119.4, 114.4)
- added D11: SK6812MINI, LED_SMD:LED_SK6812MINI_PLCC4_3.5x3.5mm_P1.75mm, F.Cu at (138.8, 82.3)
- added D12: SK6812MINI, LED_SMD:LED_SK6812MINI_PLCC4_3.5x3.5mm_P1.75mm, F.Cu at (109.9, 133.3)
- added D13: SK6812MINI, LED_SMD:LED_SK6812MINI_PLCC4_3.5x3.5mm_P1.75mm, F.Cu at (100.3, 114.4)
- added D14: SK6812MINI, LED_SMD:LED_SK6812MINI_PLCC4_3.5x3.5mm_P1.75mm, F.Cu at (81.3, 114.3)
- added D15: SK6812MINI, LED_SMD:LED_SK6812MINI_PLCC4_3.5x3.5mm_P1.75mm, F.Cu at (81.3, 95.2)
- added D16: SK6812MINI, LED_SMD:LED_SK6812MINI_PLCC4_3.5x3.5mm_P1.75mm, F.Cu at (90.9, 133.3)
- added D17: SK6812MINI, LED_SMD:LED_SK6812MINI_PLCC4_3.5x3.5mm_P1.75mm, F.Cu at (119.4, 95.5)
- moved D10 44.7 mm to (100.3, 95.2)
- moved D11 35.5 mm to (100.6, 76.2)
- renumbered D2 to D10, D1 to D11
Routing:
- net Col2: track 81.0 -> 250.8 mm, vias 1 -> 9
- net GND: track 159.0 -> 313.1 mm, vias 6 -> 17
- net Net-(D11-VDD): track 0.00 -> 139.1 mm, vias 0 -> 2
- net Net-(D16-DOUT): track 0.00 -> 70.6 mm, vias 0 -> 4
- net +5V: track 103.3 -> 171.3 mm, vias 7 -> 17
- net Net-(D15-DOUT): track 0.00 -> 51.0 mm
- net Net-(D10-DOUT): track 0.00 -> 24.7 mm, vias 0 -> 2
- net Net-(D14-DOUT): track 0.00 -> 20.2 mm, vias 0 -> 2
- net Net-(D12-DOUT): track 0.00 -> 19.7 mm
- net Net-(D13-DOUT): track 0.00 -> 16.2 mm, vias 0 -> 2
- net Net-(D1-DOUT): track 12.5 -> 26.9 mm, vias 0 -> 4
- net Net-(D1-A): track 111.1 -> 113.1 mm
- net Net-(D5-A): track 100.7 -> 102.1 mm
- net Net-(D8-A): track 90.9 -> 92.1 mm
- net ROW1: track 101.9 -> 102.9 mm
