File: project, schematic, and pcb files/hackpad.kicad_sch (KiCad schematic)
At the start: 34 parts, among them J1 Conn_01x04_Pin, SW1 SW_Push, SW10 RotaryEncoder_Switch, SW11 RotaryEncoder_Switch, SW2 SW_Push, SW3 SW_Push, SW4 SW_Push, SW5 SW_Push, SW6 SW_Push, SW7 SW_Push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

Commit message: Add files via upload
Parts:
- added D12, D13, D14, D15, D16, D17, D18: SK6812MINI, LED_SMD:LED_SK6812MINI_PLCC4_3.5x3.5mm_P1.75mm, symbol LED:SK6812MINI
- D10, D11: footprint Diode_THT:D_DO-35_SOD27_P7.62mm_Horizontal -> LED_SMD:LED_SK6812MINI_PLCC4_3.5x3.5mm_P1.75mm
Connections:
- net GND: now also D12.2 (VSS), D13.2 (VSS), D14.2 (VSS), D15.2 (VSS), D16.2 (VSS), D17.2 (VSS), D18.2 (VSS)
- net at D11.3 (DIN): now also D18.1 (DOUT); no longer D10.1 (DOUT)
- net at C2.1, C3.1, D11.4 (VDD): now also D12.4 (VDD), D13.4 (VDD), D14.4 (VDD), D15.4 (VDD), D16.4 (VDD), D17.4 (VDD), D18.4 (VDD)
- new net: D17.1 (DOUT), D18.3 (DIN)
- new net: D16.1 (DOUT), D17.3 (DIN)
- new net: D15.1 (DOUT), D16.3 (DIN)
- new net: D10.1 (DOUT), D12.3 (DIN)
- new net: D13.1 (DOUT), D14.3 (DIN)
- new net: D12.1 (DOUT), D13.3 (DIN)
- new net: D14.1 (DOUT), D15.3 (DIN)
Other:
- moved on the sheet: D11, SW11
